Commit message: edit

File: description/robot_core.xacro (robot description, xacro)
@@ -1,4 +1,17 @@
 <?xml version="1.0"?>
-<robot xmlns:xacro="http://www.ros.org/wiki/xacro">
-    ... all our links and joints will go in here ...
+<robot xmlns:xacro="http://www.ros.org/wiki/xacro" >
+    <material name="white">
+        <color rgba="1 1 1 1"/>
+    </material>
+    <material name="orange">
+        <color rgba="1 0.3 0.1 1"/>
+    </material>
+    <material name="blue">
+        <color rgba="0.2 0.2 1 1"/>
+    </material>
+    <material name="black">
+        <color rgba="0 0 0 1"/>
+    </material>
+    <!-- BASE LINK -->
+    <!-- CHASSIS LINK -->
 </robot>

Commit message: edit

File: description/robot_core.xacro (robot description, xacro)
@@ -14,4 +14,23 @@
     </material>
     <!-- BASE LINK -->
+    <link name="base_link">
+    </link>
     <!-- CHASSIS LINK -->
+    <joint name="chassis_joint" type="fixed">
+       <parent link="base_link"/>
+        <child link="chassis"/>
+        <origin xyz="-0.1 0 0"/>
+    </joint>
+    <link name="chassis">
+        <visual>
+            <origin xyz="0.15 0 0.075" rpy="0 0 0"/>
+            <geometry>
+                <box size="0.3 0.3 0.15"/>
+            </geometry>
+            <material name="white"/>
+        </visual>
+    </link>
+    <!-- LEFT WHEEL LINK -->
+    <!-- RIGHT WHEEL LINK -->
+    <!-- CASTER WHEEL LINK -->
 </robot>

Commit message: edit

File: description/robot_core.xacro (robot description, xacro)
@@ -32,5 +32,46 @@
     </link>
     <!-- LEFT WHEEL LINK -->
+    <joint name="left_wheel_joint" type="continuous">
+        <parent link="base_link"/>
+        <child link="left_wheel"/>
+        <origin xyz="0 0.175 0" rpy="-${pi/2} 0 0"/>
+        <axis xyz="0 0 1"/>
+    </joint>
+    <link name="left_wheel">
+        <visual>
+            <geometry>
+                <cylinder length="0.04" radius="0.05" />/>
+            </geometry>
+            <material name="blue"/>
+        </visual>
+    </link>
     <!-- RIGHT WHEEL LINK -->
+    <joint name="right_wheel_joint" type="continuous">
+        <parent link="base_link"/>
+        <child link="right_wheel"/>
+        <origin xyz="0 -0.175 0" rpy="${pi/2} 0 0"/>
+        <axis xyz="0 0 -1"/>
+    </joint>
+    <link name="right_wheel">
+        <visual>
+            <geometry>
+                <cylinder length="0.04" radius="0.05" />/>
+            </geometry>
+            <material name="blue"/>
+        </visual>
+    </link>
     <!-- CASTER WHEEL LINK -->
+    <joint name="caster_wheel_joint" type="fixed">
+        <parent link="chassis"/>
+        <child link="caster_wheel"/>
+        <origin xyz="0.24 0 0" rpy="0 0 0"/>
+    </joint>
+    <link name="caster_wheel">
+        <visual>
+            <geometry>
+                <sphere radius="0.05" />
+            </geometry>
+            <material name="black"/>
+        </visual>
+    </link>
 </robot>

Commit message: edit

File: description/robot_core.xacro (robot description, xacro)
@@ -30,4 +30,10 @@
             <material name="white"/>
         </visual>
+        <collision>
+            <origin xyz="0.15 0 0.075" rpy="0 0 0"/>
+            <geometry>
+                <box size="0.3 0.3 0.15"/>
+            </geometry>
+        </collision>
     </link>
     <!-- LEFT WHEEL LINK -->

Commit message: edit

File: description/robot_core.xacro (robot description, xacro)
@@ -51,4 +51,9 @@
             <material name="blue"/>
         </visual>
+        <collision>
+            <geometry>
+                <cylinder length="0.04" radius="0.05" />/>
+            </geometry>
+        </collision>
     </link>
     <!-- RIGHT WHEEL LINK -->
@@ -66,4 +71,9 @@
             <material name="blue"/>
         </visual>
+        <collision>
+            <geometry>
+                <cylinder length="0.04" radius="0.05" />/>
+            </geometry>
+        </collision>
     </link>
     <!-- CASTER WHEEL LINK -->
@@ -80,4 +90,9 @@
             <material name="black"/>
         </visual>
+        <collision>
+            <geometry>
+                <sphere radius="0.05" />
+            </geometry>
+        </collision>
     </link>
 </robot>

Commit message: edit

File: description/robot_core.xacro (robot description, xacro)
@@ -47,5 +47,5 @@
         <visual>
             <geometry>
-                <cylinder length="0.04" radius="0.05" />/>
+                <cylinder length="0.04" radius="0.05" />
             </geometry>
             <material name="blue"/>
@@ -53,5 +53,5 @@
         <collision>
             <geometry>
-                <cylinder length="0.04" radius="0.05" />/>
+                <cylinder length="0.04" radius="0.05" />
             </geometry>
         </collision>
@@ -67,5 +67,5 @@
         <visual>
             <geometry>
-                <cylinder length="0.04" radius="0.05" />/>
+                <cylinder length="0.04" radius="0.05" />
             </geometry>
             <material name="blue"/>
@@ -73,5 +73,5 @@
         <collision>
             <geometry>
-                <cylinder length="0.04" radius="0.05" />/>
+                <cylinder length="0.04" radius="0.05" />
             </geometry>
         </collision>

Commit message: edit

File: description/robot_core.xacro (robot description, xacro)
@@ -1,4 +1,5 @@
 <?xml version="1.0"?>
 <robot xmlns:xacro="http://www.ros.org/wiki/xacro" >
+    <xacro:include filename="inertial_macros.xacro" />
     <material name="white">
         <color rgba="1 1 1 1"/>
@@ -36,4 +37,7 @@
             </geometry>
         </collision>
+        <xacro:inertial_box mass="0.5" x="0.3" y="0.3" z="0.15">
+            <origin xyz="0.15 0 0.075" rpy="0 0 0"/>
+        </xacro:inertial_box>
     </link>
     <!-- LEFT WHEEL LINK -->
@@ -56,4 +60,7 @@
             </geometry>
         </collision>
+        <xacro:inertial_cylinder mass="0.1" length="0.05" radius="0.05">
+            <origin xyz="0 0 0" rpy="0 0 0"/>
+        </xacro:inertial_cylinder>
     </link>
     <!-- RIGHT WHEEL LINK -->
@@ -76,4 +83,7 @@
             </geometry>
         </collision>
+        <xacro:inertial_sphere mass="0.1" radius="0.05">
+            <origin xyz="0 0 0" rpy="0 0 0"/>
+        </xacro:inertial_sphere>
     </link>
     <!-- CASTER WHEEL LINK -->
@@ -95,4 +105,7 @@
             </geometry>
         </collision>
+       <xacro:inertial_sphere mass="0.1" radius="0.05">
+            <origin xyz="0 0 0" rpy="0 0 0"/>
+        </xacro:inertial_sphere>
     </link>
 </robot>

Commit message: edit

File: description/robot_core.xacro (robot description, xacro)
@@ -1,5 +1,5 @@
 <?xml version="1.0"?>
-<robot xmlns:xacro="http://www.ros.org/wiki/xacro" >
-    <xacro:include filename="inertial_macros.xacro" />
+<robot xmlns:xacro="http://www.ros.org/wiki/xacro">
+    <xacro:include filename="inertial_macros.xacro"/>
     <material name="white">
         <color rgba="1 1 1 1"/>
@@ -51,5 +51,5 @@
         <visual>
             <geometry>
-                <cylinder length="0.04" radius="0.05" />
+                <cylinder length="0.04" radius="0.05"/>
             </geometry>
             <material name="blue"/>
@@ -57,5 +57,5 @@
         <collision>
             <geometry>
-                <cylinder length="0.04" radius="0.05" />
+                <cylinder length="0.04" radius="0.05"/>
             </geometry>
         </collision>
@@ -74,5 +74,5 @@
         <visual>
             <geometry>
-                <cylinder length="0.04" radius="0.05" />
+                <cylinder length="0.04" radius="0.05"/>
             </geometry>
             <material name="blue"/>
@@ -80,5 +80,5 @@
         <collision>
             <geometry>
-                <cylinder length="0.04" radius="0.05" />
+                <cylinder length="0.04" radius="0.05"/>
             </geometry>
         </collision>

Commit message: edit

File: description/robot_core.xacro (robot description, xacro)
@@ -41,4 +41,7 @@
         </xacro:inertial_box>
     </link>
+    <gazebo reference="chassis">
+        <material>Gazebo/White</material>
+    </gazebo>
     <!-- LEFT WHEEL LINK -->
     <joint name="left_wheel_joint" type="continuous">
@@ -64,4 +67,7 @@
         </xacro:inertial_cylinder>
     </link>
+    <gazebo reference="chassis">
+        <material>Gazebo/Blue</material>
+    </gazebo>
     <!-- RIGHT WHEEL LINK -->
     <joint name="right_wheel_joint" type="continuous">
@@ -87,4 +93,7 @@
         </xacro:inertial_sphere>
     </link>
+    <gazebo reference="chassis">
+        <material>Gazebo/Blue</material>
+    </gazebo>
     <!-- CASTER WHEEL LINK -->
     <joint name="caster_wheel_joint" type="fixed">
@@ -109,3 +118,6 @@
         </xacro:inertial_sphere>
     </link>
+    <gazebo reference="chassis">
+        <material>Gazebo/Black</material>
+    </gazebo>
 </robot>

Commit message: edit

File: description/robot_core.xacro (robot description, xacro)
@@ -19,5 +19,5 @@
     <!-- CHASSIS LINK -->
     <joint name="chassis_joint" type="fixed">
-       <parent link="base_link"/>
+        <parent link="base_link"/>
         <child link="chassis"/>
         <origin xyz="-0.1 0 0"/>

Commit message: edit

File: description/robot_core.xacro (robot description, xacro)
@@ -25,5 +25,5 @@
     <link name="chassis">
         <visual>
-            <origin xyz="0.15 0 0.075" rpy="0 0 0"/>
+            <origin xyz="0.15 0 0.075"/>
             <geometry>
                 <box size="0.3 0.3 0.15"/>
@@ -32,5 +32,5 @@
         </visual>
         <collision>
-            <origin xyz="0.15 0 0.075" rpy="0 0 0"/>
+            <origin xyz="0.15 0 0.075"/>
             <geometry>
                 <box size="0.3 0.3 0.15"/>
@@ -54,5 +54,5 @@
         <visual>
             <geometry>
-                <cylinder length="0.04" radius="0.05"/>
+                <cylinder radius="0.05" length="0.04"/>
             </geometry>
             <material name="blue"/>
@@ -60,5 +60,5 @@
         <collision>
             <geometry>
-                <cylinder length="0.04" radius="0.05"/>
+                <cylinder radius="0.05" length="0.04"/>
             </geometry>
         </collision>
@@ -80,5 +80,5 @@
         <visual>
             <geometry>
-                <cylinder length="0.04" radius="0.05"/>
+                <cylinder radius="0.05" length="0.04"/>
             </geometry>
             <material name="blue"/>
@@ -86,8 +86,8 @@
         <collision>
             <geometry>
-                <cylinder length="0.04" radius="0.05"/>
+                <cylinder radius="0.05" length="0.04"/>
             </geometry>
         </collision>
-        <xacro:inertial_sphere mass="0.1" radius="0.05">
+        <xacro:inertial_cylinder mass="0.1" length="0.04" radius="0.05">
             <origin xyz="0 0 0" rpy="0 0 0"/>
         </xacro:inertial_sphere>
@@ -105,5 +105,5 @@
         <visual>
             <geometry>
-                <sphere radius="0.05" />
+                <sphere radius="0.05"/>
             </geometry>
             <material name="black"/>
@@ -111,8 +111,8 @@
         <collision>
             <geometry>
-                <sphere radius="0.05" />
+                <sphere radius="0.05"/>
             </geometry>
         </collision>
-       <xacro:inertial_sphere mass="0.1" radius="0.05">
+        <xacro:inertial_sphere mass="0.1" radius="0.05">
             <origin xyz="0 0 0" rpy="0 0 0"/>
         </xacro:inertial_sphere>

Commit message: edit

File: description/robot_core.xacro (robot description, xacro)
@@ -25,5 +25,5 @@
     <link name="chassis">
         <visual>
-            <origin xyz="0.15 0 0.075"/>
+            <origin xyz="0.15 0 0.075" rpy="0 0 0"/>
             <geometry>
                 <box size="0.3 0.3 0.15"/>
@@ -54,5 +54,5 @@
         <visual>
             <geometry>
-                <cylinder radius="0.05" length="0.04"/>
+                <cylinder length="0.04" radius="0.05"/>
             </geometry>
             <material name="blue"/>
@@ -60,5 +60,5 @@
         <collision>
             <geometry>
-                <cylinder radius="0.05" length="0.04"/>
+                <cylinder length="0.04" radius="0.05"/>
             </geometry>
         </collision>
@@ -80,5 +80,5 @@
         <visual>
             <geometry>
-                <cylinder radius="0.05" length="0.04"/>
+                <cylinder length="0.04" radius="0.05"/>
             </geometry>
             <material name="blue"/>
@@ -86,5 +86,5 @@
         <collision>
             <geometry>
-                <cylinder radius="0.05" length="0.04"/>
+                <cylinder length="0.04" radius="0.05"/>
             </geometry>
         </collision>

Commit message: edit

File: description/robot_core.xacro (robot description, xacro)
@@ -60,5 +60,5 @@
         <collision>
             <geometry>
-                <cylinder length="0.04" radius="0.05"/>
+                <sphere length="0.04" radius="0.05"/>
             </geometry>
         </collision>
@@ -86,5 +86,5 @@
         <collision>
             <geometry>
-                <cylinder length="0.04" radius="0.05"/>
+                <sphere length="0.04" radius="0.05"/>
             </geometry>
         </collision>

Commit message: edit

File: description/robot_core.xacro (robot description, xacro)
@@ -1,7 +1,7 @@
 <?xml version="1.0"?>
-<robot xmlns:xacro="http://www.ros.org/wiki/xacro">
+<robot xmlns:xacro="http://www.ros.org/wiki/xacro" >
     <xacro:include filename="inertial_macros.xacro"/>
     <material name="white">
-        <color rgba="1 1 1 1"/>
+        <color rgba="1 1 1 1" />
     </material>
     <material name="orange">
@@ -25,5 +25,5 @@
     <link name="chassis">
         <visual>
-            <origin xyz="0.15 0 0.075" rpy="0 0 0"/>
+            <origin xyz="0.15 0 0.075"/>
             <geometry>
                 <box size="0.3 0.3 0.15"/>
@@ -41,12 +41,9 @@
         </xacro:inertial_box>
     </link>
-    <gazebo reference="chassis">
-        <material>Gazebo/White</material>
-    </gazebo>
     <!-- LEFT WHEEL LINK -->
     <joint name="left_wheel_joint" type="continuous">
         <parent link="base_link"/>
         <child link="left_wheel"/>
-        <origin xyz="0 0.175 0" rpy="-${pi/2} 0 0"/>
+        <origin xyz="0 0.175 0" rpy="-${pi/2} 0 0" />
         <axis xyz="0 0 1"/>
     </joint>
@@ -54,5 +51,5 @@
         <visual>
             <geometry>
-                <cylinder length="0.04" radius="0.05"/>
+                <cylinder radius="0.05" length="0.04"/>
             </geometry>
             <material name="blue"/>
@@ -60,19 +57,16 @@
         <collision>
             <geometry>
-                <sphere length="0.04" radius="0.05"/>
+                <cylinder radius="0.05" length="0.04"/>
             </geometry>
         </collision>
-        <xacro:inertial_cylinder mass="0.1" length="0.05" radius="0.05">
+        <xacro:inertial_cylinder mass="0.1" length="0.04" radius="0.05">
             <origin xyz="0 0 0" rpy="0 0 0"/>
         </xacro:inertial_cylinder>
     </link>
-    <gazebo reference="left_wheel">
-        <material>Gazebo/Blue</material>
-    </gazebo>
     <!-- RIGHT WHEEL LINK -->
     <joint name="right_wheel_joint" type="continuous">
         <parent link="base_link"/>
         <child link="right_wheel"/>
-        <origin xyz="0 -0.175 0" rpy="${pi/2} 0 0"/>
+        <origin xyz="0 -0.175 0" rpy="${pi/2} 0 0" />
         <axis xyz="0 0 -1"/>
     </joint>
@@ -80,5 +74,5 @@
         <visual>
             <geometry>
-                <cylinder length="0.04" radius="0.05"/>
+                <cylinder radius="0.05" length="0.04"/>
             </geometry>
             <material name="blue"/>
@@ -86,19 +80,16 @@
         <collision>
             <geometry>
-                <sphere length="0.04" radius="0.05"/>
+                <cylinder radius="0.05" length="0.04"/>
             </geometry>
         </collision>
         <xacro:inertial_cylinder mass="0.1" length="0.04" radius="0.05">
             <origin xyz="0 0 0" rpy="0 0 0"/>
-        </xacro:inertial_sphere>
+        </xacro:inertial_cylinder>
     </link>
-    <gazebo reference="right_wheel">
-        <material>Gazebo/Blue</material>
-    </gazebo>
     <!-- CASTER WHEEL LINK -->
     <joint name="caster_wheel_joint" type="fixed">
         <parent link="chassis"/>
         <child link="caster_wheel"/>
-        <origin xyz="0.24 0 0" rpy="0 0 0"/>
+        <origin xyz="0.24 0 0"/>
     </joint>
     <link name="caster_wheel">
@@ -118,8 +109,3 @@
         </xacro:inertial_sphere>
     </link>
-    <gazebo reference="caster_wheel">
-        <material>Gazebo/Black</material>
-        <mu1 value="0.001"/>
-        <mu2 value="0.001"/>
-    </gazebo>
 </robot>
